Commit message: created environment

File: panda_ros2_gazebo/urdf/panda.urdf.xacro (robot description, xacro)
@@ -84,5 +84,5 @@
         <origin xyz="0 0 0" rpy=" 0 0 0"/>
         <geometry>
-          <box size = "0.2 0.2 1.3"/>
+          <box size = "0.2 0.2 0.7"/>
         </geometry>
       </collision>
@@ -90,5 +90,5 @@
         <origin xyz="0 0 0" rpy=" 0 0 0"/>
         <geometry>
-          <box size = "0.2 0.2 1.3"/>
+          <box size = "0.2 0.2 0.7"/>
         </geometry>
         <material name="red">
@@ -103,10 +103,10 @@
       <parent link="world" />
       <child link = "panda_base" />
-      <origin xyz="0.0 0.0 0.65" rpy="0.0 0.0 0.0" />
+      <origin xyz="0.0 0.0 0.35" rpy="0.0 0.0 0.0" />
     </joint>
     <joint name="panda_joint" type="fixed">
       <parent link="panda_base" />
       <child link = "panda_link0" />
-      <origin xyz="0.0 0.0 0.655" rpy="0.0 0.0 0.0" />
+      <origin xyz="0.0 0.0 0.35" rpy="0.0 0.0 0.0" />
     </joint>
   </xacro:if>
